File: KiCAD/Router-Board/Router-Board.sch (KiCad schematic (older format))
At the start: 41 parts, among them J2 Conn_01x14_Male, J3 Conn_01x14_Male, U1 ADG2128, U10 LME49726MY/NOPB, U11 LME49726MY/NOPB, U12 LME49726MY/NOPB, U2 LME49726MY/NOPB, U3 DS1881E-050+, U4 DS1881E-050+, U5 DS1881E-050+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

Commit message: Example improvements. Fixing library rename mistake.
Parts:
- U1: symbol VianSonus2.0-parts:ADG2128 -> ViamSonus2.0-parts:ADG2128
- U10, U11, U12, U2, U9: symbol VianSonus2.0-parts:OpAmp-Dual-Single-Symbol -> ViamSonus2.0-parts:OpAmp-Dual-Single-Symbol
- U3, U4, U5, U6, U7, U8: symbol VianSonus2.0-parts:DS1881E-050+ -> ViamSonus2.0-parts:DS1881E-050+
Changed lines of the file:
@@
 $EndDescr
 $Comp
-L VianSonus2.0-parts:ADG2128 U1
+L ViamSonus2.0-parts:ADG2128 U1
 U 1 1 5D183CD4
 P 4500 2000
@@
 $EndComp
 $Comp
-L VianSonus2.0-parts:DS1881E-050+ U3
+L ViamSonus2.0-parts:DS1881E-050+ U3
 U 1 1 5D183D42
 P 8400 1150
@@
 	9350 4500 9250 4500
 $Comp
-L VianSonus2.0-parts:OpAmp-Dual-Single-Symbol U11
+L ViamSonus2.0-parts:OpAmp-Dual-Single-Symbol U11
 U 1 1 5D193945
 P 1550 3200
@@
 GND
 $Comp
-L VianSonus2.0-parts:DS1881E-050+ U4
+L ViamSonus2.0-parts:DS1881E-050+ U4
 U 1 1 5D25BF82
 P 8400 2500
@@
 $EndComp
 $Comp
-L VianSonus2.0-parts:DS1881E-050+ U5
+L ViamSonus2.0-parts:DS1881E-050+ U5
 U 1 1 5D25C00E
 P 8400 3850
@@
 $EndComp
 $Comp
-L VianSonus2.0-parts:DS1881E-050+ U6
+L ViamSonus2.0-parts:DS1881E-050+ U6
 U 1 1 5D25C2F4
 P 9800 1150
@@
 $EndComp
 $Comp
-L VianSonus2.0-parts:DS1881E-050+ U7
+L ViamSonus2.0-parts:DS1881E-050+ U7
 U 1 1 5D262D79
 P 9800 2500
@@
 $EndComp
 $Comp
-L VianSonus2.0-parts:DS1881E-050+ U8
+L ViamSonus2.0-parts:DS1881E-050+ U8
 U 1 1 5D262F49
 P 9800 3850
@@
 	4550 950  4550 1000
 $Comp
-L VianSonus2.0-parts:OpAmp-Dual-Single-Symbol U10
+L ViamSonus2.0-parts:OpAmp-Dual-Single-Symbol U10
 U 1 1 5D6A3513
 P 1550 2050
@@
 Connection ~ 2100 2250
 $Comp
-L VianSonus2.0-parts:OpAmp-Dual-Single-Symbol U9
+L ViamSonus2.0-parts:OpAmp-Dual-Single-Symbol U9
 U 1 1 5D6B380A
 P 1550 900
@@
 Connection ~ 2100 1100
 $Comp
-L VianSonus2.0-parts:OpAmp-Dual-Single-Symbol U12
+L ViamSonus2.0-parts:OpAmp-Dual-Single-Symbol U12
 U 1 1 5D6ECE41
 P 1550 4350
@@
 ANAGND
 $Comp
-L VianSonus2.0-parts:OpAmp-Dual-Single-Symbol U2
+L ViamSonus2.0-parts:OpAmp-Dual-Single-Symbol U2
 U 1 1 5D9DA108
 P 3900 3750
