File: KiCAD/Basic-Connector-Board/Basic-Connector-Board.sch (KiCad schematic (older format))
At the start: 56 parts, among them J1 AudioJack3_Ground_Switch, J10 AudioJack3_Ground_Switch, J11 Conn_01x14_Male, J12 Conn_01x14_Male, J2 AudioJack3_Ground_Switch, J3 AudioJack3_Ground_Switch, J4 AudioJack3_Ground_Switch, J5 AudioJack3_Ground_Switch, J6 AudioJack3_Ground_Switch, J7 AudioJack3_Ground_Switch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

Commit message: Changing output cap values for better low-end response.
Parts:
- removed C1, C11, C12, C13, C14, C2, C4: 2.2uF, Capacitor_SMD:CP_Elec_6.3x5.4_Nichicon, symbol Device:CP1
- added C? (x7): 100uF, Capacitor_SMD:CP_Elec_6.3x5.4_Nichicon, symbol Device:CP1
- added J? (x2): Conn_01x04, symbol Connector_Generic:Conn_01x04
- C3: value 2.2uF -> 100uF; Digikey_Number 493-17492-1-ND -> 493-16090-1-ND; Manu_Number UUQ1H2R2MCL1GB -> UUQ0J101MCL1GB

Commit message: Adding regulator to connector board. Input-side circuit is now correct.
Parts:
- added C21, C22: 10uF, Capacitor_SMD:CP_Elec_4x5.4, symbol Device:CP1
- added J15: Barrel_Jack, symbol Connector:Barrel_Jack
- added R25, R26: 2k2, Resistor_SMD:R_0603_1608Metric, symbol Device:R
- added U1: LM1085, Package_TO_SOT_SMD:TO-263-3_TabPin2, symbol ViamSonus2.0-parts:LM1085
- C10, C15, C16, C17, C18, C19, C20, C5, C6, C7, C8, C9: value 2.2uF -> 3.3uF; footprint Capacitor_SMD:CP_Elec_6.3x5.4_Nichicon -> Capacitor_SMD:CP_Elec_4x5.4; Digikey_Number 493-17492-1-ND -> 493-17493-1-ND; Manu_Number UUQ1H2R2MCL1GB -> UUQ1H3R3MCL1GB
- J13, J14: renamed from J?; footprint (none) -> Connector_PinHeader_2.54mm:PinHeader_1x04_P2.54mm_Horizontal
- gave numbers to parts that had none: 7
Connections:
- wire segments 136 -> 165
