File: KiCAD/Basic-Connector-Board/Basic-Connector-Board.sch (KiCad schematic (older format))
At the start: 64 parts, among them J1 AudioJack3_Ground_Switch, J10 AudioJack3_Ground_Switch, J11 Conn_01x14_Male, J12 Conn_01x14_Male, J13 Conn_01x04, J14 Conn_01x04, J15 Barrel_Jack, J2 AudioJack3_Ground_Switch, J3 AudioJack3_Ground_Switch, J4 AudioJack3_Ground_Switch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

Commit message: Connector board work.
Parts:
- removed J15: Barrel_Jack, symbol Connector:Barrel_Jack
- added C23, C24: 100uF, Capacitor_SMD:CP_Elec_6.3x5.4_Nichicon, symbol Device:CP1
- added J15: 6.5 - 20v, Footprints:PJ-063AH, symbol Connector:Barrel_Jack_MountingPin
- added R27, R28, R29, R30, R31, R32, R33, R34, R35, R36, R37, R38: 2k, Resistor_SMD:R_0603_1608Metric, symbol Device:R
- added R39, R40, R41, R42, R43, R44: 20k, Resistor_SMD:R_0603_1608Metric, symbol Device:R
- J1, J10, J2, J3, J4, J5, J6, J7, J8, J9: footprint (none) -> Footprints:SJ2-3593D-SMT-TR; Digikey_Number (none) -> CP-SJ2-3593D-SMT-CT-ND; Manu_Name (none) -> CUI Devices; Manu_Number (none) -> SJ2-3593D-SMT-TR
- R25, R26: value 2k2 -> 2k; Digikey_Number RNCP0603FTD20K0CT-ND -> RNCP0603FTD2K00CT-ND; Manu_Number RNCP0603FTD20K0 -> RNCP0603FTD2K00
Connections:
- net labels added: VIn+, VIn-
- wire segments 165 -> 211
Other:
- note added: "This schematic will ensure proper operation of the zero-cross detection, and keep channel currents within\nsafe limits while mixing 5v peak-to-peak signals."

Commit message: More hardware work. More work on channel groups.
Parts:
- added J16, J17, J18, J19: Conn_01x01, MountingHole:MountingHole_3.2mm_M3_ISO14580_Pad, symbol Connector_Generic:Conn_01x01
Connections:
- wire segments 211 -> 218
Changed lines of the file:
@@
 	1    0    0    -1
 $EndComp
+$Comp
+L Connector_Generic:Conn_01x01 J16
+U 1 1 5DEE27FF
+P 6850 650
+F 0 "J16" H 6930 692 50  0000 L CNN
+F 1 "Conn_01x01" H 6930 601 50  0000 L CNN
+F 2 "MountingHole:MountingHole_3.2mm_M3_ISO14580_Pad" H 6850 650 50  0001 C CNN
+F 3 "~" H 6850 650 50  0001 C CNN
+	1    6850 650
+	1    0    0    -1
+$EndComp
+$Comp
+L Connector_Generic:Conn_01x01 J17
+U 1 1 5DEE2AA3
+P 6850 800
+F 0 "J17" H 6930 842 50  0000 L CNN
+F 1 "Conn_01x01" H 6930 751 50  0000 L CNN
+F 2 "MountingHole:MountingHole_3.2mm_M3_ISO14580_Pad" H 6850 800 50  0001 C CNN
+F 3 "~" H 6850 800 50  0001 C CNN
+	1    6850 800
+	1    0    0    -1
+$EndComp
+$Comp
+L Connector_Generic:Conn_01x01 J18
+U 1 1 5DEE2B61
+P 6850 950
+F 0 "J18" H 6930 992 50  0000 L CNN
+F 1 "Conn_01x01" H 6930 901 50  0000 L CNN
+F 2 "MountingHole:MountingHole_3.2mm_M3_ISO14580_Pad" H 6850 950 50  0001 C CNN
+F 3 "~" H 6850 950 50  0001 C CNN
+	1    6850 950
+	1    0    0    -1
+$EndComp
+$Comp
+L Connector_Generic:Conn_01x01 J19
+U 1 1 5DEE2C21
+P 6850 1100
+F 0 "J19" H 6930 1142 50  0000 L CNN
+F 1 "Conn_01x01" H 6930 1051 50  0000 L CNN
+F 2 "MountingHole:MountingHole_3.2mm_M3_ISO14580_Pad" H 6850 1100 50  0001 C CNN
+F 3 "~" H 6850 1100 50  0001 C CNN
+	1    6850 1100
+	1    0    0    -1
+$EndComp
+Wire Wire Line
+	6650 1100 6600 1100
+Wire Wire Line
+	6600 1100 6600 950
+Wire Wire Line
+	6600 650  6650 650
+Wire Wire Line
+	6650 800  6600 800
+Connection ~ 6600 800
+Wire Wire Line
+	6600 800  6600 650
+Wire Wire Line
+	6650 950  6600 950
+Connection ~ 6600 950
+Wire Wire Line
+	6600 950  6600 800
+Text Label 6600 950  1    39   ~ 0
+GND
 $EndSCHEMATC
