File: KiCAD/Basic-Connector-Board/Basic-Connector-Board.kicad_pcb (KiCad board)
At the start: 4 copper layers, 53 parts, among them J11 Conn_01x14_Male, J12 Conn_01x14_Male, J13 Conn_01x04, J14 Conn_01x04, U1 LM1085

Commit message: Connector board work.
Parts:
- added C23: 100uF, Capacitor_SMD:CP_Elec_6.3x5.4_Nichicon, F.Cu at (44.5, 73.9)
- added C24: 100uF, Capacitor_SMD:CP_Elec_6.3x5.4_Nichicon, F.Cu at (44.5, 81.3)
- added J1: AudioJack3_Ground_Switch, Footprints:SJ2-3593D-SMT-TR, F.Cu at (111.8, 80.8)
- added J10: AudioJack3_Ground_Switch, Footprints:SJ2-3593D-SMT-TR, F.Cu at (32.8, 23.6)
- added J15: 6.5 - 20v, Footprints:PJ-063AH, F.Cu at (23.9, 79.2)
- added J2: AudioJack3_Ground_Switch, Footprints:SJ2-3593D-SMT-TR, F.Cu at (111.8, 69.3)
- added J3: AudioJack3_Ground_Switch, Footprints:SJ2-3593D-SMT-TR, F.Cu at (111.8, 57.9)
- added J4: AudioJack3_Ground_Switch, Footprints:SJ2-3593D-SMT-TR, F.Cu at (111.8, 46.5)
- added J5: AudioJack3_Ground_Switch, Footprints:SJ2-3593D-SMT-TR, F.Cu at (111.8, 35.1)
- added J6: AudioJack3_Ground_Switch, Footprints:SJ2-3593D-SMT-TR, F.Cu at (111.8, 23.6)
- added J7: AudioJack3_Ground_Switch, Footprints:SJ2-3593D-SMT-TR, F.Cu at (32.8, 57.9)
- added J8: AudioJack3_Ground_Switch, Footprints:SJ2-3593D-SMT-TR, F.Cu at (32.8, 46.5)
- added J9: AudioJack3_Ground_Switch, Footprints:SJ2-3593D-SMT-TR, F.Cu at (32.8, 35.1)
- added R27: 2k, Resistor_SMD:R_0603_1608Metric, F.Cu at (83.1, 55.2)
- added R28: 2k, Resistor_SMD:R_0603_1608Metric, F.Cu at (83.1, 52.2)
- added R29: 2k, Resistor_SMD:R_0603_1608Metric, F.Cu at (83.1, 49.1)
- added R30: 2k, Resistor_SMD:R_0603_1608Metric, F.Cu at (83.1, 46.1)
- added R31: 2k, Resistor_SMD:R_0603_1608Metric, F.Cu at (83.1, 43.0)
- added R32: 2k, Resistor_SMD:R_0603_1608Metric, F.Cu at (83.1, 40.0)
- added R33: 2k, Resistor_SMD:R_0603_1608Metric, F.Cu at (83.1, 36.9)
- added R34: 2k, Resistor_SMD:R_0603_1608Metric, F.Cu at (83.1, 33.9)
- added R35: 2k, Resistor_SMD:R_0603_1608Metric, F.Cu at (83.1, 30.8)
- added R36: 2k, Resistor_SMD:R_0603_1608Metric, F.Cu at (83.1, 27.8)
- added R37: 2k, Resistor_SMD:R_0603_1608Metric, F.Cu at (83.1, 24.7)
- added R38: 2k, Resistor_SMD:R_0603_1608Metric, F.Cu at (83.1, 21.7)
- added R39: 20k, Resistor_SMD:R_0603_1608Metric, F.Cu at (71.1, 39.1)
- added R40: 20k, Resistor_SMD:R_0603_1608Metric, F.Cu at (71.1, 37.6)
- added R41: 20k, Resistor_SMD:R_0603_1608Metric, F.Cu at (71.1, 36.1)
- added R42: 20k, Resistor_SMD:R_0603_1608Metric, F.Cu at (71.1, 34.5)
- added R43: 20k, Resistor_SMD:R_0603_1608Metric, F.Cu at (71.1, 33.0)
- added R44: 20k, Resistor_SMD:R_0603_1608Metric, F.Cu at (71.1, 31.5)
- R25, R26: value 2k2 -> 2k
- moved J13 34.9 mm to (100.3, 75.2)
- moved U1 33.4 mm to (66.5, 79.2)
- moved C21 33.2 mm to (53.8, 76.5)
- moved C22 33.2 mm to (53.8, 81.8)
- moved C19 31.1 mm to (88.6, 24.9)
- moved C20 30.9 mm to (94.7, 22.6)
- moved C17 30.7 mm to (88.6, 30.7)
- moved C18 30.5 mm to (94.7, 28.4)
- moved C15 30.3 mm to (88.6, 36.6)
- moved C16 30.2 mm to (94.7, 34.3)
- moved C9 29.9 mm to (88.6, 42.4)
- moved C10 29.8 mm to (94.7, 40.1)
- moved C7 29.5 mm to (88.6, 48.3)
- moved C8 29.4 mm to (94.7, 46.0)
- moved C5 29.2 mm to (88.6, 54.1)
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Connections:
- net Net-(C21-Pad1) renamed /VIn+
- C1 pad 2: (no net) -> Net-(C1-Pad2)
- C10 pad 1: (no net) -> Net-(C10-Pad1)
- C10 pad 2: /Biased-In-R-2 -> Net-(C10-Pad2)
- C11 pad 2: (no net) -> Net-(C11-Pad2)
- C12 pad 2: (no net) -> Net-(C12-Pad2)
- C13 pad 2: (no net) -> Net-(C13-Pad2)
- C14 pad 2: (no net) -> Net-(C14-Pad2)
- C15 pad 1: (no net) -> Net-(C15-Pad1)
- C15 pad 2: /Biased-In-L-3 -> Net-(C15-Pad2)
- C16 pad 1: (no net) -> Net-(C16-Pad1)
- C16 pad 2: /Biased-In-R-3 -> Net-(C16-Pad2)
- C17 pad 1: (no net) -> Net-(C17-Pad1)
- C17 pad 2: /Biased-In-L-4 -> Net-(C17-Pad2)
- C18 pad 1: (no net) -> Net-(C18-Pad1)
- C18 pad 2: /Biased-In-R-4 -> Net-(C18-Pad2)
- C19 pad 1: (no net) -> Net-(C19-Pad1)
- C19 pad 2: /Biased-In-L-5 -> Net-(C19-Pad2)
- C2 pad 2: (no net) -> Net-(C2-Pad2)
- C20 pad 1: (no net) -> Net-(C20-Pad1)
- C20 pad 2: /Biased-In-R-5 -> Net-(C20-Pad2)
- C3 pad 2: (no net) -> Net-(C3-Pad2)
- C4 pad 2: (no net) -> Net-(C4-Pad2)
- C5 pad 1: (no net) -> Net-(C5-Pad1)
- C5 pad 2: /Biased-In-L-0 -> Net-(C5-Pad2)
- C6 pad 1: (no net) -> Net-(C6-Pad1)
- C6 pad 2: /Biased-In-R-0 -> Net-(C6-Pad2)
- C7 pad 1: (no net) -> Net-(C7-Pad1)
- C7 pad 2: /Biased-In-L-1 -> Net-(C7-Pad2)
- C8 pad 1: (no net) -> Net-(C8-Pad1)
- C8 pad 2: /Biased-In-R-1 -> Net-(C8-Pad2)
- C9 pad 1: (no net) -> Net-(C9-Pad1)
- C9 pad 2: /Biased-In-L-2 -> Net-(C9-Pad2)
- R1 pad 2: /Biased-In-L-0 -> Net-(C5-Pad2)
- R10 pad 2: /Biased-In-R-1 -> Net-(C8-Pad2)
- R11 pad 2: /Biased-In-R-2 -> Net-(C10-Pad2)
- R12 pad 2: /Biased-In-R-2 -> Net-(C10-Pad2)
- R13 pad 2: /Biased-In-L-3 -> Net-(C15-Pad2)
- R14 pad 2: /Biased-In-L-3 -> Net-(C15-Pad2)
- R15 pad 2: /Biased-In-L-4 -> Net-(C17-Pad2)
- R16 pad 2: /Biased-In-L-4 -> Net-(C17-Pad2)
- R17 pad 2: /Biased-In-L-5 -> Net-(C19-Pad2)
- R18 pad 2: /Biased-In-L-5 -> Net-(C19-Pad2)
- R19 pad 2: /Biased-In-R-3 -> Net-(C16-Pad2)
- R2 pad 2: /Biased-In-L-0 -> Net-(C5-Pad2)
- R20 pad 2: /Biased-In-R-3 -> Net-(C16-Pad2)
- R21 pad 2: /Biased-In-R-4 -> Net-(C18-Pad2)
- R22 pad 2: /Biased-In-R-4 -> Net-(C18-Pad2)
- R23 pad 2: /Biased-In-R-5 -> Net-(C20-Pad2)
- R24 pad 2: /Biased-In-R-5 -> Net-(C20-Pad2)
- R3 pad 2: /Biased-In-L-1 -> Net-(C7-Pad2)
- R4 pad 2: /Biased-In-L-1 -> Net-(C7-Pad2)
- R5 pad 2: /Biased-In-L-2 -> Net-(C9-Pad2)
- R6 pad 2: /Biased-In-L-2 -> Net-(C9-Pad2)
- R7 pad 2: /Biased-In-R-0 -> Net-(C6-Pad2)
- R8 pad 2: /Biased-In-R-0 -> Net-(C6-Pad2)
- R9 pad 2: /Biased-In-R-1 -> Net-(C8-Pad2)
Routing:
- net /Biased-In-L-0: track 0.00 -> 19.7 mm, vias 0 -> 1
- net /Biased-In-R-0: track 0.00 -> 19.5 mm, vias 0 -> 1
- net /Biased-In-L-1: track 0.00 -> 19.3 mm, vias 0 -> 1
- net /Biased-In-R-1: track 0.00 -> 19.1 mm, vias 0 -> 1
- net /Biased-In-L-2: track 0.00 -> 18.9 mm, vias 0 -> 1
- net /Biased-In-R-2: track 0.00 -> 18.7 mm, vias 0 -> 1
- net /Biased-In-L-3: track 0.00 -> 18.4 mm, vias 0 -> 1
- net /Biased-In-R-3: track 0.00 -> 18.2 mm, vias 0 -> 1
- net /Biased-In-R-5: track 0.00 -> 18.2 mm, vias 0 -> 1
- net /Biased-In-L-4: track 0.00 -> 18.0 mm, vias 0 -> 1
- net /Biased-In-L-5: track 0.00 -> 18.0 mm, vias 0 -> 1
- net /Biased-In-R-4: track 0.00 -> 17.8 mm, vias 0 -> 1
- net Net-(J5-PadRN): track 0.00 -> 16.6 mm
- net Net-(J4-PadRN): track 0.00 -> 15.8 mm
- net Net-(J3-PadRN): track 0.00 -> 15.8 mm
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Other:
- board outline added: 98 x 70.1 mm
- net class 300mA added: clearance 0.2, trace_width 0.4, via_dia 0.7, via_drill 0.254
- board text removed: "GNDD VccD"

Commit message: More hardware work. More work on channel groups.
Parts:
- added J16: Conn_01x01, MountingHole:MountingHole_3.2mm_M3_ISO14580_Pad, F.Cu at (134.0, 19.7)
- added J17: Conn_01x01, MountingHole:MountingHole_3.2mm_M3_ISO14580_Pad, F.Cu at (134.0, 25.8)
- added J18: Conn_01x01, MountingHole:MountingHole_3.2mm_M3_ISO14580_Pad, F.Cu at (140.1, 19.7)
- added J19: Conn_01x01, MountingHole:MountingHole_3.2mm_M3_ISO14580_Pad, F.Cu at (140.1, 25.8)
- moved J15 0.51 mm to (23.4, 79.2)
Other:
- board size 98 x 70.1 mm -> 97.5 x 70.6 mm
Changed lines of the file:
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@@
   (general
     (thickness 1.6)
-    (drawings 16)
+    (drawings 21)
     (tracks 131)
     (zones 0)
-    (modules 84)
+    (modules 88)
     (nets 69)
   )
@@
     (47 F.CrtYd user)
     (48 B.Fab user hide)
-    (49 F.Fab user hide)
+    (49 F.Fab user)
   )
   (setup
@@
   )
   (module Footprints:PJ-063AH (layer F.Cu)
-    (at 23.876 79.248 90)
+    (at 23.368 79.248 90)
     (fp_text reference J15 (at 0.4 8.4 90) (layer F.SilkS)
       (effects (font (size 1 1) (thickness 0.15)))
@@
     (pad "" np_thru_hole circle (at 0 3 90) (size 1.6 1.6) (drill 1.6) (layers *.Cu *.Mask))
   )
+  (module MountingHole:MountingHole_3.2mm_M3_ISO14580_Pad (layer F.Cu)
+    (at 134.004002 19.714)
+    (descr "Mounting Hole 3.2mm, M3, ISO14580")
+    (tags "mounting hole 3.2mm m3 iso14580")
+    (attr virtual)
+    (fp_text reference J16 (at 0 -3.75) (layer F.SilkS)
+      (effects (font (size 1 1) (thickness 0.15)))
+    )
+    (fp_text value Conn_01x01 (at 0 3.75) (layer F.Fab)
+      (effects (font (size 1 1) (thickness 0.15)))
+    )
+    (fp_text user %R (at 0.3 0) (layer F.Fab)
+      (effects (font (size 1 1) (thickness 0.15)))
+    )
+    (fp_circle (center 0 0) (end 2.75 0) (layer Cmts.User) (width 0.15))
+    (fp_circle (center 0 0) (end 3 0) (layer F.CrtYd) (width 0.05))
+    (pad 1 thru_hole circle (at 0 0) (size 5.5 5.5) (drill 3.2) (layers *.Cu *.Mask)
+      (net 26 /GND))
+  )
+  (module MountingHole:MountingHole_3.2mm_M3_ISO14580_Pad (layer F.Cu)
+    (at 134.004002 25.764)
+    (descr "Mounting Hole 3.2mm, M3, ISO14580")
+    (tags "mounting hole 3.2mm m3 iso14580")
+    (attr virtual)
+    (fp_text reference J17 (at 0 -3.75) (layer F.SilkS)
+      (effects (font (size 1 1) (thickness 0.15)))
+    )
+    (fp_text value Conn_01x01 (at 0 3.75) (layer F.Fab)
+      (effects (font (size 1 1) (thickness 0.15)))
+    )
+    (fp_circle (center 0 0) (end 3 0) (layer F.CrtYd) (width 0.05))
+    (fp_circle (center 0 0) (end 2.75 0) (layer Cmts.User) (width 0.15))
+    (fp_text user %R (at 0.3 0) (layer F.Fab)
+      (effects (font (size 1 1) (thickness 0.15)))
+    )
+    (pad 1 thru_hole circle (at 0 0) (size 5.5 5.5) (drill 3.2) (layers *.Cu *.Mask)
+      (net 26 /GND))
+  )
+  (module MountingHole:MountingHole_3.2mm_M3_ISO14580_Pad (layer F.Cu)
+    (at 140.054002 19.714)
+    (descr "Mounting Hole 3.2mm, M3, ISO14580")
+    (tags "mounting hole 3.2mm m3 iso14580")
+    (attr virtual)
+    (fp_text reference J18 (at 0 -3.75) (layer F.SilkS)
+      (effects (font (size 1 1) (thickness 0.15)))
+    )
+    (fp_text value Conn_01x01 (at 0 3.75) (layer F.Fab)
+      (effects (font (size 1 1) (thickness 0.15)))
+    )
+    (fp_circle (center 0 0) (end 3 0) (layer F.CrtYd) (width 0.05))
+    (fp_circle (center 0 0) (end 2.75 0) (layer Cmts.User) (width 0.15))
+    (fp_text user %R (at 0.3 0) (layer F.Fab)
+      (effects (font (size 1 1) (thickness 0.15)))
+    )
+    (pad 1 thru_hole circle (at 0 0) (size 5.5 5.5) (drill 3.2) (layers *.Cu *.Mask)
+      (net 26 /GND))
+  )
+  (module MountingHole:MountingHole_3.2mm_M3_ISO14580_Pad (layer F.Cu)
+    (at 140.054002 25.764)
+    (descr "Mounting Hole 3.2mm, M3, ISO14580")
+    (tags "mounting hole 3.2mm m3 iso14580")
+    (attr virtual)
+    (fp_text reference J19 (at 0 -3.75) (layer F.SilkS)
+      (effects (font (size 1 1) (thickness 0.15)))
+    )
+    (fp_text value Conn_01x01 (at 0 3.75) (layer F.Fab)
+      (effects (font (size 1 1) (thickness 0.15)))
+    )
+    (fp_text user %R (at 0.3 0) (layer F.Fab)
+      (effects (font (size 1 1) (thickness 0.15)))
+    )
+    (fp_circle (center 0 0) (end 2.75 0) (layer Cmts.User) (width 0.15))
+    (fp_circle (center 0 0) (end 3 0) (layer F.CrtYd) (width 0.05))
+    (pad 1 thru_hole circle (at 0 0) (size 5.5 5.5) (drill 3.2) (layers *.Cu *.Mask)
+      (net 26 /GND))
+  )
+  (gr_line (start 23.368 85.344) (end 23.368 85.852) (angle 90) (layer Edge.Cuts) (width 0.15))
+  (gr_line (start 23.368 84.328) (end 23.368 85.344) (angle 90) (layer Edge.Cuts) (width 0.15))
+  (gr_line (start 24.892 87.376) (end 119.38 87.376) (angle 90) (layer Edge.Cuts) (width 0.15))
+  (gr_line (start 23.368 18.288) (end 23.368 84.328) (angle 90) (layer Edge.Cuts) (width 0.15))
+  (gr_line (start 24.892 16.764) (end 25.4 16.764) (angle 90) (layer Edge.Cuts) (width 0.15))
   (gr_line (start 119.38 16.764) (end 25.4 16.764) (angle 90) (layer Edge.Cuts) (width 0.15))
+  (gr_arc (start 119.38 85.852) (end 120.904 85.852) (angle 90) (layer Edge.Cuts) (width 0.15))
+  (gr_arc (start 24.892 85.852) (end 24.892 87.376) (angle 90) (layer Edge.Cuts) (width 0.15))
+  (gr_arc (start 24.892 18.288) (end 23.368 18.288) (angle 90) (layer Edge.Cuts) (width 0.15))
+  (gr_arc (start 119.38 18.288) (end 119.38 16.764) (angle 90) (layer Edge.Cuts) (width 0.15))
   (gr_line (start 120.904 85.344) (end 120.904 18.288) (angle 90) (layer Edge.Cuts) (width 0.15))
-  (gr_arc (start 119.38 18.2626) (end 119.38 16.7386) (angle 90) (layer Edge.Cuts) (width 0.15))
-  (gr_arc (start 24.384 84.4296) (end 24.384 85.9536) (angle 90) (layer Edge.Cuts) (width 0.15))
-  (gr_arc (start 119.38 85.3186) (end 120.904 85.3186) (angle 90) (layer Edge.Cuts) (width 0.15))
-  (gr_arc (start 25.019 18.2626) (end 23.495 18.2626) (angle 90) (layer Edge.Cuts) (width 0.15))
   (gr_line (start 65.024 56.7436) (end 101.092 56.7436) (angle 90) (layer F.SilkS) (width 0.15))
   (gr_line (start 102.616 55.2196) (end 102.616 21.6916) (angle 90) (layer F.SilkS) (width 0.15))
